File: elec/layout/default/ma732.kicad_pcb (KiCad board)
At the start: 2 copper layers, 225.7 x 100.8 mm, 0 parts

Commit message: update layout
Parts:
- added C1: 25V 1uF X5R ±10% 0402 Multilayer Ceramic Capacitors MLCC - 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, lib:C0402, F.Cu at (156.6, 87.2)
- added U1: , lib:VQFN-16_L3.0-W3.0-P0.50-BL-EP1.6, F.Cu at (159.2, 88.5)
Routing:
- net vcc: track 0.00 -> 1.21 mm
Changed lines of the file:
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@@
   )
   (net 0 "")
+  (net 1 "gnd")
+  (net 2 "vcc-4")
+  (net 3 "sck")
+  (net 4 "n_c")
+  (net 5 "vcc")
+  (net 6 "sclk")
+  (net 7 "mgl")
+  (net 8 "pwm")
+  (net 9 "miso")
+  (net 10 "vcc-2")
+  (net 11 "cs")
+  (net 12 "mosi")
+  (net 13 "vcc-3")
+  (net 14 "vcc-1")
+  (net 15 "ssd")
+  (footprint "lib:VQFN-16_L3.0-W3.0-P0.50-BL-EP1.6" (layer "F.Cu")
+    (at 159.235 88.545)
+    (attr smd)
+    (fp_text reference "U1" (at 0 -5.5) (layer "F.SilkS")
+        (effects (font (size 1 1) (thickness 0.15)))
+    )
+    (fp_text value "" (at 0 5.5) (layer "F.Fab")
+        (effects (font (size 1 1) (thickness 0.15)))
+    )
+    (fp_text user "${REFERENCE}" (at 0 0) (layer "F.Fab")
+        (effects (font (size 1 1) (thickness 0.15)))
+    )
+    (fp_line (start -1.5 -1.5) (end -1.5 -1.04)
+      (stroke (width 0.1) (type solid)) (layer "F.SilkS"))
+    (fp_line (start -1.5 -1.5) (end -1.05 -1.5)
+      (stroke (width 0.1) (type solid)) (layer "F.SilkS"))
+    (fp_line (start -1.5 1.04) (end -1.5 1.5)
+      (stroke (width 0.1) (type solid)) (layer "F.SilkS"))
+    (fp_line (start -1.5 1.5) (end -1.05 1.5)
+      (stroke (width 0.1) (type solid)) (layer "F.SilkS"))
+    (fp_line (start 1.04 -1.5) (end 1.5 -1.5)
+      (stroke (width 0.1) (type solid)) (layer "F.SilkS"))
+    (fp_line (start 1.04 1.5) (end 1.5 1.5)
+      (stroke (width 0.1) (type solid)) (layer "F.SilkS"))
+    (fp_line (start 1.5 -1.04) (end 1.5 -1.5)
+      (stroke (width 0.1) (type solid)) (layer "F.SilkS"))
+    (fp_line (start 1.5 1.5) (end 1.5 1.04)
+      (stroke (width 0.1) (type solid)) (layer "F.SilkS"))
+    (fp_arc (start -1.25 1.74) (mid -1.245 1.75866) (end -1.25866 1.745)
+      (stroke (width 0.25) (type solid)) (layer "F.SilkS"))
+    (fp_circle (center -0.75 1.75) (end -0.65 1.75)
+      (stroke (width 0.2) (type solid)) (fill none) (layer "Cmts.User"))
+    (fp_circle (center -1.5 1.5) (end -1.47 1.5)
+      (stroke (width 0.06) (type solid)) (fill none) (layer "F.Fab"))
+    (pad "1" smd rect (at -0.75 1.5) (size 0.28 0.8) (layers "F.Cu" "F.Paste" "F.Mask")
+      (net 15 "ssd") (pintype "stereo"))
+    (pad "2" smd rect (at -0.25 1.5) (size 0.28 0.8) (layers "F.Cu" "F.Paste" "F.Mask")
+      (net 14 "vcc-1") (pintype "stereo"))
+    (pad "3" smd rect (at 0.25 1.5) (size 0.28 0.8) (layers "F.Cu" "F.Paste" "F.Mask")
+      (net 13 "vcc-3") (pintype "stereo"))
+    (pad "4" smd rect (at 0.75 1.5) (size 0.28 0.8) (layers "F.Cu" "F.Paste" "F.Mask")
+      (net 12 "mosi") (pintype "stereo"))
+    (pad "5" smd rect (at 1.5 0.75) (size 0.8 0.28) (layers "F.Cu" "F.Paste" "F.Mask")
+      (net 11 "cs") (pintype "stereo"))
+    (pad "6" smd rect (at 1.5 0.25) (size 0.8 0.28) (layers "F.Cu" "F.Paste" "F.Mask")
+      (net 10 "vcc-2") (pintype "stereo"))
+    (pad "7" smd rect (at 1.5 -0.25) (size 0.8 0.28) (layers "F.Cu" "F.Paste" "F.Mask")
+      (net 9 "miso") (pintype "stereo"))
+    (pad "8" smd rect (at 1.5 -0.75) (size 0.8 0.28) (layers "F.Cu" "F.Paste" "F.Mask")
+      (net 1 "gnd") (pintype "stereo"))
+    (pad "9" smd rect (at 0.75 -1.5) (size 0.28 0.8) (layers "F.Cu" "F.Paste" "F.Mask")
+      (net 8 "pwm") (pintype "stereo"))
+    (pad "10" smd rect (at 0.25 -1.5) (size 0.28 0.8) (layers "F.Cu" "F.Paste" "F.Mask")
+      (net 1 "gnd") (pintype "stereo"))
+    (pad "11" smd rect (at -0.25 -1.5) (size 0.28 0.8) (layers "F.Cu" "F.Paste" "F.Mask")
+      (net 7 "mgl") (pintype "stereo"))
+    (pad "12" smd rect (at -0.75 -1.5) (size 0.28 0.8) (layers "F.Cu" "F.Paste" "F.Mask")
+      (net 6 "sclk") (pintype "stereo"))
+    (pad "13" smd rect (at -1.5 -0.75) (size 0.8 0.28) (layers "F.Cu" "F.Paste" "F.Mask")
+      (net 5 "vcc") (pintype "stereo"))
+    (pad "14" smd rect (at -1.5 -0.25) (size 0.8 0.28) (layers "F.Cu" "F.Paste" "F.Mask")
+      (net 4 "n_c") (pintype "stereo"))
+    (pad "15" smd rect (at -1.5 0.25) (size 0.8 0.28) (layers "F.Cu" "F.Paste" "F.Mask")
+      (net 3 "sck") (pintype "stereo"))
+    (pad "16" smd rect (at -1.5 0.75) (size 0.8 0.28) (layers "F.Cu" "F.Paste" "F.Mask")
+      (net 2 "vcc-4") (pintype "stereo"))
+    (pad "17" smd rect (at 0 0 90) (size 1.6 1.6) (layers "F.Cu" "F.Paste" "F.Mask")
+      (net 1 "gnd") (pintype "stereo"))
+    (model "/Users/narayanpowderly/Documents/atopile-workspace/servo-drive/.ato/modules/ma732/elec/footprints/footprints.3dshapes/VQFN-16_L3.0-W3.0-H1.0-P0.50.wrl"
+      (offset (xyz -0 -0.05 -0))
+      (scale (xyz 1 1 1))
+      (rotate (xyz 0 0 270))
+    )
+  )
+  (footprint "lib:C0402" (layer "F.Cu")
+    (at 156.569325 87.212516 90)
+    (descr "Capacitor SMD 0402 (1005 Metric), square (rectangular) end terminal, IPC_7351 nominal, (Body size source: IPC-SM-782 page 76, https://www.pcb-3d.com/wordpress/wp-content/uploads/ipc-sm-782a_amendment_1_and_2.pdf), generated with kicad-footprint-generator")
+    (tags "capacitor")
+    (attr smd)
+    (fp_text reference "C1" (at 0 -1.16 90) (layer "F.SilkS")
+        (effects (font (size 1 1) (thickness 0.15)))
+    )
+    (fp_text value "25V 1uF X5R ±10% 0402  Multilayer Ceramic Capacitors MLCC - SMD/SMT ROHS" (at 0 1.16 90) (layer "F.Fab")
+        (effects (font (size 1 1) (thickness 0.15)))
+    )
+    (fp_text user "${REFERENCE}" (at 0 0 90) (layer "F.Fab")
+        (effects (font (size 0.25 0.25) (thickness 0.04)))
+    )
+    (fp_line (start -0.107836 -0.36) (end 0.107836 -0.36)
+      (stroke (width 0.12) (type solid)) (layer "F.SilkS"))
+    (fp_line (start -0.107836 0.36) (end 0.107836 0.36)
+      (stroke (width 0.12) (type solid)) (layer "F.SilkS"))
+    (fp_line (start -0.91 -0.46) (end 0.91 -0.46)
+      (stroke (width 0.05) (type solid)) (layer "F.CrtYd"))
+    (fp_line (start -0.91 0.46) (end -0.91 -0.46)
+      (stroke (width 0.05) (type solid)) (layer "F.CrtYd"))
+    (fp_line (start 0.91 -0.46) (end 0.91 0.46)
+      (stroke (width 0.05) (type solid)) (layer "F.CrtYd"))
+    (fp_line (start 0.91 0.46) (end -0.91 0.46)
+      (stroke (width 0.05) (type solid)) (layer "F.CrtYd"))
+    (fp_line (start -0.5 -0.25) (end 0.5 -0.25)
+      (stroke (width 0.1) (type solid)) (layer "F.Fab"))
+    (fp_line (start -0.5 0.25) (end -0.5 -0.25)
+      (stroke (width 0.1) (type solid)) (layer "F.Fab"))
+    (fp_line (start 0.5 -0.25) (end 0.5 0.25)
+      (stroke (width 0.1) (type solid)) (layer "F.Fab"))
+    (fp_line (start 0.5 0.25) (end -0.5 0.25)
+      (stroke (width 0.1) (type solid)) (layer "F.Fab"))
+    (pad "1" smd roundrect (at -0.48 0 90) (size 0.56 0.62) (layers "F.Cu" "F.Paste" "F.Mask") (roundrect_rratio 0.25)
+      (net 5 "vcc") (pintype "stereo"))
+    (pad "2" smd roundrect (at 0.48 0 90) (size 0.56 0.62) (layers "F.Cu" "F.Paste" "F.Mask") (roundrect_rratio 0.25)
+      (net 1 "gnd") (pintype "stereo"))
+    (model "${KICAD6_3DMODEL_DIR}/Capacitor_SMD.3dshapes/C_0402_1005Metric.wrl"
+      (offset (xyz 0 0 0))
+      (scale (xyz 1 1 1))
+      (rotate (xyz 0 0 0))
+    )
+  )
   (gr_circle (center 225.62 81.79) (end 227.32 81.79)
     (stroke (width 0.1) (type solid)) (fill none) (layer "Edge.Cuts"))
@@
       (xy 69.100734 49.778315)
     )
-    (stroke (width 0) (type solid)) (fill none) (layer "Edge.Cuts"))
+    (stroke (width 0.1) (type solid)) (fill none) (layer "Edge.Cuts"))
   (gr_arc (start 261.62 113.79) (mid 260.448427 116.618427) (end 257.62 117.79)
     (stroke (width 0.1) (type solid)) (layer "Edge.Cuts"))
@@
     (effects (font (size 2 2) (thickness 0.1)) (justify left bottom))
   )
+  (segment (start 157.735 87.795) (end 156.671809 87.795) (width 0.25) (layer "F.Cu") (net 5))
+  (segment (start 156.671809 87.795) (end 156.569325 87.692516) (width 0.25) (layer "F.Cu") (net 5))
   (group "" (id 6c1ef9f7-0f34-47bb-ac1a-76df23fb396e)
     (members
